Commit message: Fix wrong file paths

File: rover_demo_gz/urdf/macros.xacro (robot description, xacro)
@@ -21,10 +21,10 @@
         <visual>
           <geometry>
-            <mesh filename="package://rover_demo_gz/models/leo/Rocker.dae"/>
+            <mesh filename="package://leo/Rocker.dae"/>
           </geometry>
         </visual>
         <collision>
           <geometry>
-            <mesh filename="package://rover_demo_gz/models/leo/Rocker_outline.stl"/>
+            <mesh filename="package://leo/Rocker_outline.stl"/>
           </geometry>
         </collision>
@@ -43,5 +43,5 @@
         <visual>
           <geometry>
-            <mesh filename="package://rover_demo_gz/models/leo/Wheel${model}.dae"/>
+            <mesh filename="package://leo/Wheel${model}.dae"/>
           </geometry>
         </visual>
@@ -60,5 +60,5 @@
         <collision>
           <geometry>
-            <mesh filename="package://rover_demo_gz/models/leo/Wheel_outline.stl"/>
+            <mesh filename="package://leo/Wheel_outline.stl"/>
           </geometry>
         </collision>
@@ -77,5 +77,5 @@
         <visual>
           <geometry>
-            <mesh filename="package://rover_demo_gz/models/leo/WheelMecanum${model}.dae"/>
+            <mesh filename="package://leo/WheelMecanum${model}.dae"/>
           </geometry>
         </visual>
@@ -88,5 +88,5 @@
         <collision>
           <geometry>
-            <mesh filename="package://rover_demo_gz/models/leo/Mecanum_wheel_outline.stl"/>
+            <mesh filename="package://leo/Mecanum_wheel_outline.stl"/>
           </geometry>
         </collision>
@@ -109,10 +109,10 @@
       <visual>
         <geometry>
-          <mesh filename="package://rover_demo_gz/models/leo/Chassis.dae"/>
+          <mesh filename="package://leo/Chassis.dae"/>
         </geometry>
       </visual>
       <collision>
         <geometry>
-          <mesh filename="package://rover_demo_gz/models/leo/Chassis_outline.stl"/>
+          <mesh filename="package://leo/Chassis_outline.stl"/>
         </geometry>
       </collision>
@@ -144,5 +144,5 @@
         <visual>
           <geometry>
-            <mesh filename="package://rover_demo_gz/models/leo/Antenna.dae"/>
+            <mesh filename="package://leo/Antenna.dae"/>
           </geometry>
         </visual>
