Commit message: Fixed rtabnav for leo rover

File: rover_demo_gz/urdf/drone.urdf.xacro (robot description, xacro)
@@ -4,5 +4,5 @@
   <xacro:property name="mass" value="1.0"/>
   <xacro:property name="arm_length" value="0.25"/>
-  <xacro:property name="link_prefix" value = "" />
+  <xacro:property name="link_prefix" value = "drone/" />
   <xacro:arg name="robot_ns" default=""/>
   <xacro:property name="robot_ns" value="$(arg robot_ns)"/>
@@ -188,5 +188,5 @@
         <update_frequency>10</update_frequency>
         <odom_topic>${robot_ns}/true_pose</odom_topic>
-        <odom_frame>world</odom_frame>
+        <odom_frame>odom</odom_frame>
         <robot_base_frame>${link_prefix}base_link</robot_base_frame>
         <tf_topic>tf</tf_topic>

File: rover_demo_gz/urdf/macros.xacro (robot description, xacro)
@@ -415,12 +415,11 @@
           <friction>
             <ode>
-              <mu>15</mu>
+              <mu>1</mu>
               <mu2>1</mu2>
-              <slip1>0</slip1>
-              <slip2>0</slip2>
-              <fdir1>1 0 0</fdir1>
-            </ode>
-            <bullet>
-              <friction>15</friction>
+              <slip1>0.01</slip1>
+              <slip2>0.01</slip2>
+            </ode>
+            <bullet>
+              <friction>1</friction>
               <friction2>1</friction2>
               <rolling_friction>0</rolling_friction>
@@ -435,12 +434,11 @@
           <friction>
             <ode>
-              <mu>15</mu>
+              <mu>1</mu>
               <mu2>1</mu2>
-              <slip1>0</slip1>
-              <slip2>0</slip2>
-              <fdir1>1 0 0</fdir1>
-            </ode>
-            <bullet>
-              <friction>15</friction>
+              <slip1>0.01</slip1>
+              <slip2>0.01</slip2>
+            </ode>
+            <bullet>
+              <friction>1</friction>
               <friction2>1</friction2>
               <rolling_friction>0</rolling_friction>
@@ -455,12 +453,11 @@
           <friction>
             <ode>
-              <mu>15</mu>
+              <mu>1</mu>
               <mu2>1</mu2>
-              <slip1>0</slip1>
-              <slip2>0</slip2>
-              <fdir1>1 0 0</fdir1>
-            </ode>
-            <bullet>
-              <friction>15</friction>
+              <slip1>0.01</slip1>
+              <slip2>0.01</slip2>
+            </ode>
+            <bullet>
+              <friction>1</friction>
               <friction2>1</friction2>
               <rolling_friction>0</rolling_friction>
@@ -475,12 +472,11 @@
           <friction>
             <ode>
-              <mu>15</mu>
+              <mu>1</mu>
               <mu2>1</mu2>
-              <slip1>0</slip1>
-              <slip2>0</slip2>
-              <fdir1>1 0 0</fdir1>
-            </ode>
-            <bullet>
-              <friction>15</friction>
+              <slip1>0.01</slip1>
+              <slip2>0.01</slip2>
+            </ode>
+            <bullet>
+              <friction>1</friction>
               <friction2>1</friction2>
               <rolling_friction>0</rolling_friction>
@@ -547,5 +543,5 @@
           </scan>
           <range>
-            <min>0.08</min>
+            <min>1.0</min>
             <max>10.0</max>
             <resolution>0.01</resolution>
@@ -603,5 +599,5 @@
         <update_frequency>10</update_frequency>
         <odom_topic>${link_prefix}true_pose</odom_topic>
-        <odom_frame>world</odom_frame>
+        <odom_frame>odom</odom_frame>
         <robot_base_frame>${link_prefix}base_footprint</robot_base_frame>
         <tf_topic>tf</tf_topic>
@@ -630,7 +626,7 @@
               />
     <xacro:if value="${fixed}">
-      <link name="world"/>
+      <link name="odom"/>
       <joint name="fixed" type="fixed">
-        <parent link="world"/>
+        <parent link="odom"/>
         <child link="${link_prefix}base_footprint"/>
         <origin xyz="0.0 0.0 1.0"/>
